Commit message: add apply_force.cpp

File: qm_description/urdf/manipulator/common/kinova_common.xacro (robot description, xacro)
@@ -15,5 +15,5 @@
 <xacro:include filename="$(find qm_description)/urdf/manipulator/common/kinova_inertial.xacro" />
     <xacro:property name="J_PI" value="3.1415926535897931" />
-    <xacro:macro name="kinova_armlink" params="link_name link_mesh ring_mesh:=ring_big use_ring_mesh:=false mesh_no col:=false">
+    <xacro:macro name="kinova_armlink" params="link_name link_mesh ring_mesh:=ring_big use_ring_mesh:=false mesh_no col:=true">
       <link name="${link_name}">
           <visual>

File: qm_description/urdf/manipulator/j2n6s300fix.xacro (robot description, xacro)
@@ -116,5 +116,5 @@
         <xacro:kinova_armlink link_name="${prefix}_link_5" link_mesh="${link_5_mesh}" use_ring_mesh="true" ring_mesh="ring_small" mesh_no="${link_5_mesh_no}"/>
         <xacro:kinova_armjoint joint_name="${prefix}_joint_5" type="${joint_5_type}" parent="${prefix}_link_4" child="${prefix}_link_5" joint_axis_xyz="${joint_5_axis_xyz}" joint_origin_xyz="${joint_5_origin_xyz}" joint_origin_rpy="${joint_5_origin_rpy}" joint_lower_limit="${joint_5_lower_limit}" joint_upper_limit="${joint_5_upper_limit}" joint_velocity_limit="${joint_5_velocity_limit}" joint_torque_limit="${joint_5_torque_limit}"/>
-        <xacro:kinova_armlink link_name="${prefix}_link_6" link_mesh="${link_6_mesh}" use_ring_mesh="true" ring_mesh="ring_small" mesh_no="${link_6_mesh_no}"/>
+        <xacro:kinova_armlink link_name="${prefix}_link_6" link_mesh="${link_6_mesh}" use_ring_mesh="true" ring_mesh="ring_small" mesh_no="${link_6_mesh_no}" />
         <xacro:kinova_armjoint joint_name="${prefix}_joint_6" type="${joint_6_type}" parent="${prefix}_link_5" child="${prefix}_link_6" joint_axis_xyz="${joint_6_axis_xyz}" joint_origin_xyz="${joint_6_origin_xyz}" joint_origin_rpy="${joint_6_origin_rpy}" joint_lower_limit="${joint_6_lower_limit}" joint_upper_limit="${joint_6_upper_limit}" joint_velocity_limit="${joint_6_velocity_limit}" joint_torque_limit="${joint_6_torque_limit}"/>
         <xacro:kinova_virtual_link link_name="${prefix}_end_effector"/>

File: qm_description/urdf/sensor/ft_sensor.xacro (robot description, xacro)
@@ -8,11 +8,11 @@
             <origin xyz="0.0 0.0 0.0" rpy="0.0 0.0 0.0"/>
         </visual>
-        <!-- <collision>
+        <collision>
             <geometry>
                 <cylinder radius="0.0375" length="0.01"/>
             </geometry>
             <origin xyz="0.0 0.0 0.0" rpy="0.0 0.0 0.0"/>
-        </collision> -->
-        <inertial>
+        </collision>
+        <!-- <inertial>
             <mass value="0.0001"/>
             <inertia ixx="3.5989583333333335E-8"
@@ -22,6 +22,6 @@
                      iyz="0.0"
                      izz="7.03125E-8"/>
-        </inertial>
-        <!-- <inertial>
+        </inertial> -->
+        <inertial>
             <mass value="0.01"/>
             <inertia ixx="7.1441E-05"
@@ -31,5 +31,5 @@
                      iyz="-8.5336E-09"
                      izz="0.00013366"/>
-        </inertial> -->
+        </inertial>
     </link>
     <joint name="ft_sensor_joint" type="revolute">
@@ -46,5 +46,5 @@
     <gazebo>
     <plugin name="ft_sensor_joint" filename="libgazebo_ros_ft_sensor.so">
-        <updateRate>1000.0</updateRate>
+        <updateRate>100.0</updateRate>
         <topicName>ft_sensor_topic</topicName>
         <jointName>ft_sensor_joint</jointName>

Commit message: add multidimensional set-valued admittance for manipulator

File: qm_description/urdf/manipulator/common/kinova_common.xacro (robot description, xacro)
@@ -15,5 +15,5 @@
 <xacro:include filename="$(find qm_description)/urdf/manipulator/common/kinova_inertial.xacro" />
     <xacro:property name="J_PI" value="3.1415926535897931" />
-    <xacro:macro name="kinova_armlink" params="link_name link_mesh ring_mesh:=ring_big use_ring_mesh:=false mesh_no col:=true">
+    <xacro:macro name="kinova_armlink" params="link_name link_mesh ring_mesh:=ring_big use_ring_mesh:=false mesh_no col:=false">
       <link name="${link_name}">
           <visual>

File: qm_description/urdf/sensor/ft_sensor.xacro (robot description, xacro)
@@ -8,10 +8,10 @@
             <origin xyz="0.0 0.0 0.0" rpy="0.0 0.0 0.0"/>
         </visual>
-        <collision>
+        <!-- <collision>
             <geometry>
                 <cylinder radius="0.0375" length="0.01"/>
             </geometry>
             <origin xyz="0.0 0.0 0.0" rpy="0.0 0.0 0.0"/>
-        </collision>
+        </collision> -->
         <!-- <inertial>
             <mass value="0.0001"/>
@@ -24,4 +24,22 @@
         </inertial> -->
         <inertial>
+            <mass value="0.00001"/>
+            <inertia ixx="3.5989583333333335E-9"
+                     ixy="0.0"
+                     ixz="0.0"
+                     iyy="3.5156250000041194E-9"
+                     iyz="0.0"
+                     izz="7.03125E-9"/>
+        </inertial>
+        <!-- <inertial>
+            <mass value="1.0E-7"/>
+            <inertia ixx="3.6E-10"
+                    ixy="0.0"
+                    ixz="0.0"
+                    iyy="3.5E-10"
+                    iyz="0.0"
+                    izz="7.0E-10"/>
+        </inertia>      -->
+        <!-- <inertial>
             <mass value="0.01"/>
             <inertia ixx="7.1441E-05"
@@ -31,5 +49,5 @@
                      iyz="-8.5336E-09"
                      izz="0.00013366"/>
-        </inertial>
+        </inertial> -->
     </link>
     <joint name="ft_sensor_joint" type="revolute">
